Commit message: mujoco

File: urdf/four_wheels_chassis.urdf (robot description, URDF)
Before this commit: robot four_wheels_chassis, 5 links, 4 joints
Links:
- link base_link: geometry collision mesh filename=meshes/base_link.STL; visual mesh filename=meshes/base_link.STL
- link wheel_lb_link: geometry collision mesh filename=meshes/wheel_lb_link.STL; visual mesh filename=meshes/wheel_lb_link.STL
- link wheel_lf_link: geometry collision mesh filename=meshes/wheel_lf_link.STL; visual mesh filename=meshes/wheel_lf_link.STL
- link wheel_rb_link: geometry collision mesh filename=meshes/wheel_rb_link.STL; visual mesh filename=meshes/wheel_rb_link.STL
- link wheel_rf_link: geometry collision mesh filename=meshes/wheel_rf_link.STL; visual mesh filename=meshes/wheel_rf_link.STL
